Commit message: Update start position

File: srdf/panda_arm.xacro (robot description, xacro)
@@ -11,13 +11,4 @@
     </group>
     <!--GROUP STATES: Purpose: Define a named state for a particular group, in terms of joint values. This is useful to define states like 'folded arms'-->
-    <group_state name="ready" group="panda_arm">
-      <joint name="panda_joint1" value="0" />
-      <joint name="panda_joint2" value="-0.785" />
-      <joint name="panda_joint3" value="0" />
-      <joint name="panda_joint4" value="-2.356" />
-      <joint name="panda_joint5" value="0" />
-      <joint name="panda_joint6" value="1.571" />
-      <joint name="panda_joint7" value="0.785" />
-    </group_state>
     <group_state name="extended" group="panda_arm">
       <joint name="panda_joint1" value="0" />
@@ -27,14 +18,5 @@
       <joint name="panda_joint5" value="0" />
       <joint name="panda_joint6" value="0" />
-      <joint name="panda_joint7" value="0.785" />
-    </group_state>
-    <group_state name="transport" group="panda_arm">
-      <joint name="panda_joint1" value="0" />
-      <joint name="panda_joint2" value="-0.5599" />
-      <joint name="panda_joint3" value="0" />
-      <joint name="panda_joint4" value="-2.97" />
-      <joint name="panda_joint5" value="0" />
-      <joint name="panda_joint6" value="0" />
-      <joint name="panda_joint7" value="0.785" />
+      <joint name="panda_joint7" value="0" />
     </group_state>
     <!--END EFFECTOR: Purpose: Represent information about an end effector.-->
